File: hw/sch_pcb/PINHOLDER02.kicad_pcb (KiCad board)
At the start: 2 copper layers, 50.3 x 30 mm, 8 parts, among them J1 HEADER_1x03, M1 HOLE, M2 HOLE, M3 HOLE, M4 HOLE

Commit message: uprava layoutu pro velkou diodu
Parts:
- removed M1: HOLE, Mlab_Mechanical:MountingHole_3mm
- moved TP1 4.13 mm to (168.7, 88.7)
- moved TP2 2.55 mm to (152.4, 88.7)
Routing:
- net Net-(J1-Pad1): track 4.28 -> 6.13 mm
Other:
- board size 50.3 x 30 mm -> 60.6 x 60.4 mm
Changed lines of the file:
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@@
       (effects (font (size 1 1) (thickness 0.15)))
     )
-    (fp_text value "HEADER_1x03" (at 0 4.87 90) (layer "F.Fab")
+    (fp_text value "HEADER_1x03" (at 0 4.87 90) (layer "F.Fab") hide
       (effects (font (size 1 1) (thickness 0.15)))
     )
@@
     )
   )
-  (footprint "Mlab_Mechanical:MountingHole_3mm" placed (layer "F.Cu")
-    (at 190.25 96.8)
-    (descr "Mounting hole, Befestigungsbohrung, 3mm, No Annular, Kein Restring,")
-    (tags "Mounting hole, Befestigungsbohrung, 3mm, No Annular, Kein Restring,")
-    (property "Sheetfile" "PINHOLDER02.kicad_sch")
-    (property "Sheetname" "")
-    (attr through_hole)
-    (fp_text reference "M1" (at 0 -4.191) (layer "F.SilkS") hide
-      (effects (font (size 1.524 1.524) (thickness 0.3048)))
-    )
-    (fp_text value "HOLE" (at 0 4.191) (layer "F.SilkS") hide
-      (effects (font (size 1.524 1.524) (thickness 0.3048)))
-    )
-    (fp_circle (center 0 0) (end 2.99974 0) (layer "F.Fab") (width 0.381) (fill none))
-    (pad "1" thru_hole circle (at 0 0) (size 6 6) (drill 3) (layers *.Cu *.Mask)
-      (net 2 "GND") (pintype "input") (clearance 1) (zone_connect 2))
-    (model "${MLAB}/src/3d/mechanical/m3_komplet.step"
-      (offset (xyz 0 0 0))
-      (scale (xyz 1 1 1))
-      (rotate (xyz 0 0 0))
-    )
-  )
   (footprint "TestPoint:TestPoint_Pad_D2.0mm" (layer "B.Cu")
     (at 148.3 83.15 180)
@@
   )
   (footprint "Mlab_CON:TestPoint_Pad_D0.5mm_noSilk" (layer "B.Cu")
-    (at 167.9 84.65 180)
+    (at 168.7 88.7 180)
     (descr "SMD pad as test Point, diameter 1.0mm")
     (tags "test point SMD pad")
@@
   )
   (footprint "TestPoint:TestPoint_Keystone_5019_Minature" (layer "B.Cu")
-    (at 154.95 88.7 90)
+    (at 152.4 88.7 90)
     (descr "SMT Test Point- Micro Miniature 5019, http://www.keyelco.com/product-pdf.cfm?p=1357")
     (tags "Test Point")
@@
     )
   )
-  (gr_line (start 144.786 101.624) (end 195.074 101.624) (layer "Edge.Cuts") (width 0.1))
-  (gr_line (start 144.786 71.656) (end 195.074 71.656) (layer "Edge.Cuts") (width 0.1))
-  (gr_line (start 195.074 71.656) (end 195.074 101.624) (layer "Edge.Cuts") (width 0.1))
-  (gr_line (start 144.786 101.624) (end 144.786 71.656) (layer "Edge.Cuts") (width 0.1))
+  (gr_line (start 144.712 132) (end 205.3 131.9) (layer "Edge.Cuts") (width 0.1))
+  (gr_line (start 144.786 71.656) (end 205.15 71.6) (layer "Edge.Cuts") (width 0.1))
+  (gr_line (start 205.15 71.6) (end 205.3 131.9) (layer "Edge.Cuts") (width 0.1))
+  (gr_line (start 144.712 132) (end 144.786 71.656) (layer "Edge.Cuts") (width 0.1))
   (gr_rect (start 134.8 78.6) (end 146.2 90.4) (layer "User.1") (width 0.15) (fill solid))
   (gr_line (start 146.6 78.2) (end 146.6 90.8) (layer "User.2") (width 1))
@@
   (gr_line (start 134.3 77.2) (end 147.3 77.2) (layer "User.4") (width 3))
   (gr_line (start 147 91) (end 134 91) (layer "User.4") (width 3))
-  (gr_text "MLAB" (at 157.274 99.474) (layer "F.Cu")
+  (gr_text "MLAB" (at 149.2 130.3) (layer "F.Cu")
     (effects (font (size 1.5 1.5) (thickness 0.3)))
   )
-  (gr_text "MLAB" (at 157.324 99.424) (layer "B.Cu")
+  (gr_text "MLAB" (at 149.2 130.3) (layer "B.Cu")
     (effects (font (size 1.5 1.5) (thickness 0.3)) (justify mirror))
   )
@@
   (segment (start 167.621 88.929) (end 167.9 88.65) (width 0.4) (layer "F.Cu") (net 1))
   (via (at 167.9 88.65) (size 0.8) (drill 0.4) (layers "F.Cu" "B.Cu") (net 1))
+  (segment (start 167.95 88.7) (end 167.9 88.65) (width 0.25) (layer "B.Cu") (net 1))
   (via (at 146.9 83.2) (size 0.8) (drill 0.4) (layers "F.Cu" "B.Cu") (net 2))
   (segment (start 146.9 83.2) (end 146.95 83.15) (width 0.25) (layer "B.Cu") (net 2))
   (segment (start 146.95 83.15) (end 148.3 83.15) (width 0.25) (layer "B.Cu") (net 2))
-  (segment (start 158.905 88.7) (end 159.134 88.929) (width 0.4) (layer "F.Cu") (net 3))
-  (segment (start 154.95 88.7) (end 158.905 88.7) (width 0.4) (layer "F.Cu") (net 3))
-  (via (at 154.95 88.7) (size 0.8) (drill 0.4) (layers "F.Cu" "B.Cu") (net 3))
+  (segment (start 158.905 88.7) (end 153.1 88.7) (width 0.4) (layer "F.Cu") (net 3))
+  (segment (start 159.134 88.929) (end 158.905 88.7) (width 0.4) (layer "F.Cu") (net 3))
+  (via (at 153.1 88.7) (size 0.8) (drill 0.4) (layers "F.Cu" "B.Cu") (net 3))
   (zone (net 2) (net_name "GND") (layer "F.Cu") (hatch edge 0.508)
     (connect_pads (clearance 0.4))
@@
     (polygon
       (pts
-        (xy 199.224 110.524)
-        (xy 129.924 110.524)
+        (xy 214.924 136.724)
+        (xy 129.924 136.724)
         (xy 129.924 57.524)
-        (xy 199.224 57.524)
+        (xy 214.924 57.524)
       )
     )
@@
     (polygon
       (pts
-        (xy 172.374 84.124)
-        (xy 172.374 89.124)
-        (xy 167.374 89.124)
-        (xy 167.374 84.124)
+        (xy 187.2 87.7)
+        (xy 187.2 105)
+        (xy 167.1 105)
+        (xy 167.1 87.7)
       )
     )
@@
     (polygon
       (pts
-        (xy 200.724 111.474)
-        (xy 131.774 111.474)
+        (xy 214.924 135.674)
+        (xy 131.774 135.674)
         (xy 131.774 59.974)
-        (xy 200.724 59.974)
+        (xy 214.924 59.974)
       )
     )
